File: hardware/pcb/projects/groove-pad-ctrl/groove-pad-ctrl.kicad_pcb (KiCad board)
At the start: 2 copper layers, 128.5 x 78 mm, 115 parts, among them J1 TOUCH_L, J2 TOUCH_R, J3 Conn_01x03, J4 Conn_01x07, J5 Conn_01x07, J6 TOUCH_LOGO, J7 Conn_01x07, J8 Conn_01x05, SW1 SW_Push, SW10 SW_Push, SW11 SW_Push, SW12 SW_Push, SW13 SW_Push, SW14 SW_Push, SW15 SW_Push, SW16 SW_Push, SW17 SW_Push, SW18 SW_Push, SW19 SW_Push, SW2 SW_Push, SW20 SW_Push, SW3 SW_Push, SW4 SW_Push, SW5 SW_Push, SW6 SW_Push, SW7 SW_Push, SW8 SW_Push, SW9 SW_Push, U1 STM32F303R8Tx, U2 MB85RS2MT, Y1 8MHz

Commit message: ver 0.1
Parts:
- added C12: 100n, Capacitor_SMD:C_0603_1608Metric, B.Cu at (114.2, 83.3)
- added C13: 100n, Capacitor_SMD:C_0603_1608Metric, B.Cu at (123.5, 94.6)
- added C14: 100n, Capacitor_SMD:C_0603_1608Metric, B.Cu at (117.0, 101.8)
- added C15: 100n, Capacitor_SMD:C_0603_1608Metric, B.Cu at (105.0, 95.5)
- added C16: 100n, Capacitor_SMD:C_0603_1608Metric, B.Cu at (128.6, 82.2)
- added G***: LOGO, custom:Groove_Controller_Silk, F.Cu at (114.2, 89.0)
- added G***: LOGO, symbol:logo, F.Cu at (114.2, 89.0)
- added J9: TOUCH_R_C, custom:PAD_CENTER, F.Cu at (150.2, 79.0)
- added R38: 1k, Resistor_SMD:R_0603_1608Metric, B.Cu at (135.2, 88.5)
- added REF**: MountingHole_3_3.65, custom:MountingHole_3mm_3.65mm, F.Cu at (175.6, 53.5)
- added REF**: MountingHole_3_3.65, custom:MountingHole_3mm_3.65mm, F.Cu at (53.0, 53.5)
- added REF**: MountingHole_3_3.65, custom:MountingHole_3mm_3.65mm, F.Cu at (175.6, 124.6)
- added REF**: MountingHole_3_3.65, custom:MountingHole_3mm_3.65mm, F.Cu at (53.0, 124.6)
- C1, C10, C11, C2, C3, C4, C5, C6, C7, C8, C9, FB1, FB2, J3, J4, J5, J7, J8, R10, R11, R12, R13, R14, R15, R16, R17, R18, R19, R2, R20, R24, R25, R26, R27, R28, R29, R3, R30, R31, R32, R33, R34, R35, R36, R37, R4, R5, R6, R7, R8, R9: moved to B.Cu
- D1, D10, D11, D12, D13, D14, D15, D16, D2, D3, D4, D5, D6, D7, D8, D9: footprint kicadlib:SOD-123_mod2 -> custom:SOD-123_mod2; moved to B.Cu
- J1, J2: footprint kicadlib:CassettePad -> custom:CassettePad
- J6: value TOUCH_LOGO -> TOUCH_L_C; footprint kicadlib:TEST_PAD_Small -> custom:PAD_CENTER
- R1: value 100k -> 10k; moved to B.Cu
- R21, R22, R23: value 47 -> 10k; moved to B.Cu
- SW1, SW10, SW11, SW12, SW13, SW14, SW15, SW16, SW17, SW18, SW2, SW3, SW4, SW5, SW6, SW7, SW8, SW9: footprint kicadlib:SW_PUSH_SMD -> custom:SW_Tactile_SKRH
- SW19, SW20: footprint kicadlib:SW_PUSH_SMD -> custom:SW_Tactile_SPST_Angled_ALPS_SKHLL
- U2: footprint kicadlib:MB85RS2MT -> custom:MB85RS2MT
- Y1: footprint kicadlib:Crystal_SMD_Abracon_ABM3-2pin_5.0x3.2mm_hand -> custom:Crystal_SMD_Abracon_ABM3-2pin_5.0x3.2mm_hand; moved to B.Cu
- moved C10 133.7 mm to (102.8, 58.4), turned to 270 degrees
- moved R14 130.8 mm to (169.0, 66.5), turned to 180 degrees
- moved J5 129.2 mm to (168.9, 87.0)
- moved D9 122.2 mm to (65.2, 117.0), turned to 90 degrees
- moved SW20 120.9 mm to (150.2, 53.5)
- moved FB2 119.7 mm to (99.8, 58.4), turned to 270 degrees
- moved D2 119.1 mm to (79.2, 105.0), turned to 90 degrees
- moved Y1 118.2 mm to (122.0, 82.5)
- moved D1 116.1 mm to (65.2, 105.0), turned to 90 degrees
- moved C4 115.1 mm to (58.8, 96.5)
- moved J7 112.9 mm to (106.6, 58.8), turned to 270 degrees
- moved R17 110.1 mm to (125.2, 58.0), turned to 90 degrees
- moved SW19 108.4 mm to (78.2, 53.5)
- moved FB1 107.6 mm to (58.2, 93.7), turned to 90 degrees
- moved R1 107.6 mm to (60.8, 93.5), turned to 90 degrees
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Connections:
- C7 pad 1: /G4_IO1 -> /G3_IO1
- R16 pad 1: /G4_IO2 -> /G3_IO2
- U1 pad 20: Net-(U1-Pad20) -> /BTN_1
- U1 pad 24: /BTN_1 -> /BTN_2
- U1 pad 25: /BTN_2 -> /G3_IO1
- U1 pad 26: /BTN_MINUS -> /G3_IO2
- U1 pad 27: /BTN_PLUS -> /G3_IO3
- U1 pad 28: Net-(U1-Pad28) -> /~RAM_CS
- U1 pad 29: /BTN_MODE -> /BTN_B
- U1 pad 30: /LED_MODE -> /BTN_A
- U1 pad 41: /~RAM_CS -> /BTN_MINUS
- U1 pad 42: /G4_IO1 -> Net-(U1-Pad42)
- U1 pad 43: /G4_IO2 -> Net-(U1-Pad43)
- U1 pad 44: /BTN_RUN -> /BTN_MODE
- U1 pad 45: /LED_RUN -> /LED_MODE
- U1 pad 50: /~OLED_CS -> /BTN_PLUS
- U1 pad 62: Net-(U1-Pad62) -> /~OLED_CS
- U1 pad 8: /BTN_A -> /LED_RUN
- U1 pad 9: /BTN_B -> /BTN_RUN
Routing:
- net +3V3: track 0.00 -> 440.4 mm, vias 0 -> 26
- net +3.3VA: track 0.00 -> 164.5 mm, vias 0 -> 6
- net /~RESET: track 0.00 -> 154.0 mm, vias 0 -> 2
- net /LED_1: track 0.00 -> 142.4 mm, vias 0 -> 5
- net Net-(C6-Pad1): track 0.00 -> 125.6 mm
- net /BTN_MINUS: track 0.00 -> 122.2 mm, vias 0 -> 4
- net /LED_2: track 0.00 -> 120.2 mm, vias 0 -> 5
- net /BTN_2: track 0.00 -> 117.3 mm, vias 0 -> 4
- net Net-(R33-Pad2): track 0.00 -> 117.0 mm, vias 0 -> 4
- net /BTN_3: track 0.00 -> 114.8 mm, vias 0 -> 4
- net Net-(R27-Pad2): track 0.00 -> 113.6 mm, vias 0 -> 4
- net Net-(R31-Pad2): track 0.00 -> 110.8 mm, vias 0 -> 4
- net Net-(R29-Pad2): track 0.00 -> 109.4 mm, vias 0 -> 4
- net /BTN_1: track 0.00 -> 103.3 mm, vias 0 -> 4
- net /BTN_PLUS: track 0.00 -> 100.3 mm, vias 0 -> 2
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- added copper zone on B.Cu, net GND
- added copper zone on F.Cu, net GND
Other:
- outline, holes or cut-outs redrawn
- net class Default: clearance 0.2 -> 0.19; trace_width 0.25 -> 0.2; via_dia 0.8 -> 0.6; via_drill 0.4 -> 0.3
- rule trace_clearance: 0.2 -> 0.19
- board text added: "GROOVE CONTROLLER ver0.1"

Commit message: change MCU
Parts:
- U1: value STM32F303R8Tx -> STM32F072R8Tx
Changed lines of the file:
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@@
       (effects (font (size 1 1) (thickness 0.15)) (justify mirror))
     )
-    (fp_text value STM32F303R8Tx (at 0 -7.4 225) (layer B.Fab)
+    (fp_text value STM32F072R8Tx (at 0 -7.4 225) (layer B.Fab)
       (effects (font (size 1 1) (thickness 0.15)) (justify mirror))
     )
