File: hardware/pcb/projects/groove-pad-ctrl/groove-pad-ctrl.sch (KiCad schematic (older format))
At the start: 115 parts, among them J1 TOUCH_L, J2 TOUCH_R, J3 Conn_01x03, J4 Conn_01x07, J5 Conn_01x07, J6 TOUCH_LOGO, J7 Conn_01x07, J8 Conn_01x05, SW1 SW_Push, SW10 SW_Push, SW11 SW_Push, SW12 SW_Push, SW13 SW_Push, SW14 SW_Push, SW15 SW_Push, SW16 SW_Push, SW17 SW_Push, SW18 SW_Push, SW19 SW_Push, SW2 SW_Push, SW20 SW_Push, SW3 SW_Push, SW4 SW_Push, SW5 SW_Push, SW6 SW_Push, SW7 SW_Push, SW8 SW_Push, SW9 SW_Push, U1 STM32F303R8Tx, U2 MB85RS2MT, Y1 8MHz

Commit message: ver 0.1
Parts:
- added C12, C13, C14, C15, C16: 100n, Capacitor_SMD:C_0603_1608Metric, symbol cqd_touch_pad:C_Small
- added J9: TOUCH_R_C, custom:PAD_CENTER, symbol Connector_Generic:Conn_01x01
- added R38: 1k, Resistor_SMD:R_0603_1608Metric, symbol cqd_touch_pad:R
- D1, D10, D11, D12, D13, D14, D15, D16, D2, D3, D4, D5, D6, D7, D8, D9: footprint kicadlib:SOD-123_mod2 -> custom:SOD-123_mod2
- J1, J2: footprint kicadlib:CassettePad -> custom:CassettePad
- J6: value TOUCH_LOGO -> TOUCH_L_C; footprint kicadlib:TEST_PAD_Small -> custom:PAD_CENTER
- R1: value 100k -> 10k
- R21, R22, R23: value 47 -> 10k
- SW1, SW10, SW11, SW12, SW13, SW14, SW15, SW16, SW17, SW18, SW2, SW3, SW4, SW5, SW6, SW7, SW8, SW9: footprint kicadlib:SW_PUSH_SMD -> custom:SW_Tactile_SKRH
- SW19, SW20: footprint kicadlib:SW_PUSH_SMD -> custom:SW_Tactile_SPST_Angled_ALPS_SKHLL
- U2: footprint kicadlib:MB85RS2MT -> custom:MB85RS2MT
- Y1: footprint kicadlib:Crystal_SMD_Abracon_ABM3-2pin_5.0x3.2mm_hand -> custom:Crystal_SMD_Abracon_ABM3-2pin_5.0x3.2mm_hand
Connections:
- net +3.3VA: now also C16.2
- net +3V3: now also C12.1, C13.1, C14.1, C15.1
- net BTN_1: now also U1.20 (PA4); no longer U1.24 (PC4)
- net BTN_2: now also U1.24 (PC4); no longer U1.25 (PC5)
- net BTN_A: now also U1.30 (PB11); no longer U1.8 (PC0)
- net BTN_B: now also U1.29 (PB10); no longer U1.9 (PC1)
- net BTN_MINUS: now also U1.41 (PA8); no longer U1.26 (PB0)
- net BTN_MODE: now also U1.44 (PA11); no longer U1.29 (PB10)
- net BTN_PLUS: now also U1.50 (PA15); no longer U1.27 (PB1)
- net BTN_RUN: now also U1.9 (PC1); no longer U1.44 (PA11)
- net GND: now also C12.2, C13.2, C14.2, C15.2, C16.1
- net LED_MODE: now also U1.45 (PA12); no longer U1.30 (PB11)
- net LED_RUN: now also U1.8 (PC0); no longer U1.45 (PA12)
- net ~OLED_CS: now also U1.62 (PB9); no longer U1.50 (PA15)
- net ~RAM_CS: now also U1.28 (PB2); no longer U1.41 (PA8)
- net G4_IO1: no longer names the net of U1.42 (PA9)
- net G4_IO1: no longer C7.1
- net G4_IO2: no longer names the net of U1.43 (PA10)
- net G4_IO2: no longer R16.1
- new net: J9.1 (Pin_1), R38.2
- new net G3_IO1: C7.1, U1.25 (PC5)
- new net G3_IO2: R16.1, U1.26 (PB0)
- new net G3_IO3: R38.1, U1.27 (PB1)
- no-connect marks 7 -> 6
Other:
- note added: "ALPS SKHLLCA010"
- note added: "ALPS SKRGAAD010"
- moved on the sheet: R13, R17, R18

Commit message: change MCU
Parts:
- U1: value STM32F303R8Tx -> STM32F072R8Tx; symbol MCU_ST_STM32F3:STM32F303R8Tx -> MCU_ST_STM32F0:STM32F072R8Tx
Other:
- moved on the sheet: C16
Changed lines of the file:
@@
 	7200 1500 7700 1500
 $Comp
-L MCU_ST_STM32F3:STM32F303R8Tx U1
+L MCU_ST_STM32F0:STM32F072R8Tx U1
 U 1 1 5E4EB293
 P 3150 3000
 F 0 "U1" H 3150 3050 50  0000 C CNN
-F 1 "STM32F303R8Tx" H 3150 2950 50  0000 C CNN
+F 1 "STM32F072R8Tx" H 3150 2950 50  0000 C CNN
 F 2 "Package_QFP:LQFP-64_10x10mm_P0.5mm" H 2550 1300 50  0001 R CNN
 F 3 "http://www.st.com/st-web-ui/static/active/en/resource/technical/document/datasheet/DM00092070.pdf" H 3150 3000 50  0001 C CNN
@@
 Wire Wire Line
 	2950 1100 3050 1100
-Wire Wire Line
-	3350 1100 3350 1200
 Connection ~ 2950 1100
 Wire Wire Line
@@
 Wire Wire Line
 	3250 1200 3250 1100
-Connection ~ 3250 1100
-Wire Wire Line
-	3250 1100 3350 1100
 Wire Wire Line
 	3150 1200 3150 1100
@@
 L power:+3.3VA #PWR04
 U 1 1 5E4FFAA4
-P 3450 1050
-F 0 "#PWR04" H 3450 900 50  0001 C CNN
-F 1 "+3.3VA" H 3465 1223 50  0000 C CNN
-F 2 "" H 3450 1050 50  0001 C CNN
-F 3 "" H 3450 1050 50  0001 C CNN
-	1    3450 1050
+P 3350 750
+F 0 "#PWR04" H 3350 600 50  0001 C CNN
+F 1 "+3.3VA" H 3365 923 50  0000 C CNN
+F 2 "" H 3350 750 50  0001 C CNN
+F 3 "" H 3350 750 50  0001 C CNN
+	1    3350 750
 	1    0    0    -1
 $EndComp
@@
 Connection ~ 4500 750
 Wire Wire Line
-	3450 1050 3450 1150
+	3350 750  3350 850
 $Comp
 L cqd_touch_pad:R R1
@@
 L cqd_touch_pad:C_Small C16
 U 1 1 5E515BD7
-P 3550 1150
-F 0 "C16" V 3400 1250 50  0000 L CNN
-F 1 "100n" V 3500 1200 50  0000 L CNN
-F 2 "Capacitor_SMD:C_0603_1608Metric" H 3550 1150 50  0001 C CNN
-F 3 "" H 3550 1150 50  0000 C CNN
-	1    3550 1150
+P 3450 850
+F 0 "C16" V 3300 950 50  0000 L CNN
+F 1 "100n" V 3400 900 50  0000 L CNN
+F 2 "Capacitor_SMD:C_0603_1608Metric" H 3450 850 50  0001 C CNN
+F 3 "" H 3450 850 50  0000 C CNN
+	1    3450 850
 	0    1    1    0
 $EndComp
-Connection ~ 3450 1150
-Wire Wire Line
-	3450 1150 3450 1200
+Connection ~ 3350 850
 $Comp
 L cqd_touch_pad:GND #PWR043
 U 1 1 5E5161B6
-P 3650 1150
-F 0 "#PWR043" H 3650 900 50  0001 C CNN
-F 1 "GND" H 3650 1000 50  0000 C CNN
-F 2 "" H 3650 1150 50  0000 C CNN
-F 3 "" H 3650 1150 50  0000 C CNN
-	1    3650 1150
+P 3550 850
+F 0 "#PWR043" H 3550 600 50  0001 C CNN
+F 1 "GND" H 3550 700 50  0000 C CNN
+F 2 "" H 3550 850 50  0000 C CNN
+F 3 "" H 3550 850 50  0000 C CNN
+	1    3550 850
 	1    0    0    -1
 $EndComp
@@
 Text Label 3900 3600 0    50   ~ 0
 OLED_DC
+Wire Wire Line
+	3350 850  3350 1200
+$Comp
+L power:+3.3V #PWR?
+U 1 1 5E6EDB73
+P 3450 1200
+F 0 "#PWR?" H 3450 1050 50  0001 C CNN
+F 1 "+3.3V" H 3600 1200 50  0000 C CNN
+F 2 "" H 3450 1200 50  0001 C CNN
+F 3 "" H 3450 1200 50  0001 C CNN
+	1    3450 1200
+	1    0    0    -1
+$EndComp
 $EndSCHEMATC
